Commit message: rkg0.5

File: rc_arm_stack/rc_arm_description/urdf/rc_arm_2/rc_arm_2.urdf.xacro (robot description, xacro)
@@ -71,5 +71,5 @@
     <child link="l1"/>
     <axis xyz="0 0 -1"/>
-    <limit lower="-0.2942036732051034" upper="3.9357963267948963" effort="14.0" velocity="12.0"/>
+    <limit lower="-1.8650" upper="2.3650" effort="14.0" velocity="12.0"/>
   </joint>
   <link name="l2">

File: rc_arm_stack/rc_arm_description/urdf/rc_arm_2/rc_arm_2_ros2_control.xacro (robot description, xacro)
@@ -67,6 +67,6 @@
         <param name="payload_low_stiffness_kd">${hardware_config.payload_low_stiffness_kd_j1}</param>
         <command_interface name="position">
-          <param name="min">-0.2942036732051034</param>
-          <param name="max">3.9357963267948963</param>
+          <param name="min">-1.8650</param>
+          <param name="max">2.3650</param>
         </command_interface>
         <command_interface name="velocity">

Commit message: rkg0.6 fix mujoco orientation error

File: rc_arm_stack/rc_arm_description/urdf/rc_arm_2/rc_arm_2.urdf.xacro (robot description, xacro)
@@ -71,5 +71,5 @@
     <child link="l1"/>
     <axis xyz="0 0 -1"/>
-    <limit lower="-1.8650" upper="2.3650" effort="14.0" velocity="12.0"/>
+    <limit lower="-0.2942036732051034" upper="3.9357963267948963" effort="14.0" velocity="12.0"/>
   </joint>
   <link name="l2">

File: rc_arm_stack/rc_arm_description/urdf/rc_arm_2/rc_arm_2_ros2_control.xacro (robot description, xacro)
@@ -67,6 +67,6 @@
         <param name="payload_low_stiffness_kd">${hardware_config.payload_low_stiffness_kd_j1}</param>
         <command_interface name="position">
-          <param name="min">-1.8650</param>
-          <param name="max">2.3650</param>
+          <param name="min">-0.2942036732051034</param>
+          <param name="max">3.9357963267948963</param>
         </command_interface>
         <command_interface name="velocity">

File: rc_robotarm_mujoco/assets/robots/rc_arm_2/02_SUB_RoboticArm.urdf (robot description, URDF)
Before this commit: robot 02_SUB_RoboticArm, 5 links, 4 joints
Joints:
- joint j1: origin xyz=0 -0.00169679105026498 0.0135 rpy=0 0 0 -> xyz=0 -0.00169679105026498 0.0135 rpy=0 0 1.5707963267948966
