Commit message: huge change ,big clean!!!

File: rc_moveit/rc_arm_description/urdf/rc_arm_2/rc_arm_2.urdf.xacro (robot description, xacro)
@@ -2,32 +2,5 @@
 <robot name="rc_arm_2" xmlns:xacro="http://www.ros.org/wiki/xacro">
   <xacro:arg name="use_mock_hardware" default="false"/>
-  <xacro:arg name="can_interface" default="can0"/>
-  <xacro:arg name="host_can_id" default="253"/>
-  <xacro:arg name="can_enabled" default="true"/>
-  <xacro:arg name="external_feedback_enabled" default="false"/>
-  <xacro:arg name="external_feedback_topic" default="/rc_arm_2/mujoco_joint_states"/>
-  <xacro:arg name="external_feedback_timeout" default="0.2"/>
-  <xacro:arg name="s_curve_enabled" default="true"/>
-  <xacro:arg name="scalar_path_time_enabled" default="true"/>
-  <xacro:arg name="smoothing_alpha" default="0.2"/>
-  <xacro:arg name="max_velocity" default="2.0"/>
-  <xacro:arg name="max_acceleration" default="8.0"/>
-  <xacro:arg name="max_jerk" default="50.0"/>
-  <xacro:arg name="low_stiffness_mode" default="false"/>
-  <xacro:arg name="low_stiffness_kp" default="20.0"/>
-  <xacro:arg name="low_stiffness_kd" default="2.0"/>
-  <xacro:arg name="low_stiffness_kp_j1" default="0.0"/>
-  <xacro:arg name="low_stiffness_kd_j1" default="0.0"/>
-  <xacro:arg name="low_stiffness_kp_j2" default="0.0"/>
-  <xacro:arg name="low_stiffness_kd_j2" default="0.0"/>
-  <xacro:arg name="low_stiffness_kp_j3" default="0.0"/>
-  <xacro:arg name="low_stiffness_kd_j3" default="0.0"/>
-  <xacro:arg name="low_stiffness_kp_j4" default="0.0"/>
-  <xacro:arg name="low_stiffness_kd_j4" default="0.0"/>
-  <xacro:arg name="low_stiffness_torque_bias" default="0.0"/>
-  <xacro:arg name="use_pinocchio_gravity" default="true"/>
-  <xacro:arg name="gravity_feedforward_ratio" default="1.0"/>
-  <xacro:arg name="use_pinocchio_inverse_dynamics" default="true"/>
-  <xacro:arg name="urdf_path" default="$(find rc_arm_description)/urdf/rc_arm_2/rc_arm_2.pinocchio.urdf"/>
+  <xacro:arg name="hardware_config_file" default="$(find rc_arm_description)/config/rc_arm_2/rc_arm_2_hardware.real.yaml"/>
   <xacro:include filename="rc_arm_2_ros2_control.xacro"/>
   <material name="dark_gray">
@@ -206,31 +179,4 @@
   <xacro:rc_arm_2_ros2_control
     use_mock_hardware="$(arg use_mock_hardware)"
-    can_interface="$(arg can_interface)"
-    host_can_id="$(arg host_can_id)"
-    can_enabled="$(arg can_enabled)"
-    external_feedback_enabled="$(arg external_feedback_enabled)"
-    external_feedback_topic="$(arg external_feedback_topic)"
-    external_feedback_timeout="$(arg external_feedback_timeout)"
-    s_curve_enabled="$(arg s_curve_enabled)"
-    scalar_path_time_enabled="$(arg scalar_path_time_enabled)"
-    smoothing_alpha="$(arg smoothing_alpha)"
-    max_velocity="$(arg max_velocity)"
-    max_acceleration="$(arg max_acceleration)"
-    max_jerk="$(arg max_jerk)"
-    low_stiffness_mode="$(arg low_stiffness_mode)"
-    low_stiffness_kp="$(arg low_stiffness_kp)"
-    low_stiffness_kd="$(arg low_stiffness_kd)"
-    low_stiffness_kp_j1="$(arg low_stiffness_kp_j1)"
-    low_stiffness_kd_j1="$(arg low_stiffness_kd_j1)"
-    low_stiffness_kp_j2="$(arg low_stiffness_kp_j2)"
-    low_stiffness_kd_j2="$(arg low_stiffness_kd_j2)"
-    low_stiffness_kp_j3="$(arg low_stiffness_kp_j3)"
-    low_stiffness_kd_j3="$(arg low_stiffness_kd_j3)"
-    low_stiffness_kp_j4="$(arg low_stiffness_kp_j4)"
-    low_stiffness_kd_j4="$(arg low_stiffness_kd_j4)"
-    low_stiffness_torque_bias="$(arg low_stiffness_torque_bias)"
-    use_pinocchio_gravity="$(arg use_pinocchio_gravity)"
-    gravity_feedforward_ratio="$(arg gravity_feedforward_ratio)"
-    use_pinocchio_inverse_dynamics="$(arg use_pinocchio_inverse_dynamics)"
-    urdf_path="$(arg urdf_path)"/>
+    hardware_config_file="$(arg hardware_config_file)"/>
 </robot>

File: rc_moveit/rc_arm_description/urdf/rc_arm_2/rc_arm_2_ros2_control.xacro (robot description, xacro)
@@ -1,5 +1,8 @@
 <?xml version="1.0"?>
 <robot xmlns:xacro="http://www.ros.org/wiki/xacro">
-  <xacro:macro name="rc_arm_2_ros2_control" params="use_mock_hardware can_interface host_can_id can_enabled external_feedback_enabled external_feedback_topic external_feedback_timeout s_curve_enabled scalar_path_time_enabled smoothing_alpha max_velocity max_acceleration max_jerk low_stiffness_mode low_stiffness_kp low_stiffness_kd low_stiffness_kp_j1 low_stiffness_kd_j1 low_stiffness_kp_j2 low_stiffness_kd_j2 low_stiffness_kp_j3 low_stiffness_kd_j3 low_stiffness_kp_j4 low_stiffness_kd_j4 low_stiffness_torque_bias use_pinocchio_gravity gravity_feedforward_ratio use_pinocchio_inverse_dynamics urdf_path">
+  <xacro:macro name="rc_arm_2_ros2_control" params="use_mock_hardware hardware_config_file">
+    <xacro:property name="hardware_config_path" value="${hardware_config_file}"/>
+    <xacro:property name="hardware_config" value="${xacro.load_yaml(hardware_config_path)}"/>
+    <xacro:property name="description_package_share" value="${hardware_config_path.rsplit('/config/', 1)[0]}"/>
     <ros2_control name="RcArm2System" type="system">
       <hardware>
@@ -10,27 +13,35 @@
         <xacro:unless value="${use_mock_hardware}">
           <plugin>rc_arm_hardware/RsA3HardwareInterface</plugin>
-          <param name="can_interface">${can_interface}</param>
-          <param name="host_can_id">${host_can_id}</param>
-          <param name="can_enabled">${can_enabled}</param>
-          <param name="external_feedback_enabled">${external_feedback_enabled}</param>
-          <param name="external_feedback_topic">${external_feedback_topic}</param>
-          <param name="external_feedback_timeout">${external_feedback_timeout}</param>
-          <param name="position_kp">60.0</param>
-          <param name="position_kd">3.0</param>
-          <param name="velocity_limit">8.0</param>
-          <param name="s_curve_enabled">${s_curve_enabled}</param>
-          <param name="scalar_path_time_enabled">${scalar_path_time_enabled}</param>
-          <param name="smoothing_alpha">${smoothing_alpha}</param>
-          <param name="max_velocity">${max_velocity}</param>
-          <param name="max_acceleration">${max_acceleration}</param>
-          <param name="max_jerk">${max_jerk}</param>
-          <param name="low_stiffness_mode">${low_stiffness_mode}</param>
-          <param name="low_stiffness_kp">${low_stiffness_kp}</param>
-          <param name="low_stiffness_kd">${low_stiffness_kd}</param>
-          <param name="low_stiffness_torque_bias">${low_stiffness_torque_bias}</param>
-          <param name="use_pinocchio_gravity">${use_pinocchio_gravity}</param>
-          <param name="gravity_feedforward_ratio">${gravity_feedforward_ratio}</param>
-          <param name="use_pinocchio_inverse_dynamics">${use_pinocchio_inverse_dynamics}</param>
-          <param name="urdf_path">${urdf_path}</param>
+          <param name="backend">${hardware_config.backend}</param>
+          <param name="can_interface">${hardware_config.can_interface}</param>
+          <param name="host_can_id">${hardware_config.host_can_id}</param>
+          <param name="external_feedback_topic">${hardware_config.external_feedback_topic}</param>
+          <param name="external_feedback_timeout">${hardware_config.external_feedback_timeout}</param>
+          <param name="mujoco_command_topic">${hardware_config.mujoco_command_topic}</param>
+          <param name="dm_sn">${hardware_config.dm_sn}</param>
+          <param name="dm_nom_baud">${hardware_config.dm_nom_baud}</param>
+          <param name="dm_dat_baud">${hardware_config.dm_dat_baud}</param>
+          <param name="dm_control_mode">${hardware_config.dm_control_mode}</param>
+          <param name="position_kp">${hardware_config.position_kp}</param>
+          <param name="position_kd">${hardware_config.position_kd}</param>
+          <param name="velocity_limit">${hardware_config.velocity_limit}</param>
+          <param name="s_curve_enabled">${hardware_config.s_curve_enabled}</param>
+          <param name="scalar_path_time_enabled">${hardware_config.scalar_path_time_enabled}</param>
+          <param name="smoothing_alpha">${hardware_config.smoothing_alpha}</param>
+          <param name="max_velocity">${hardware_config.max_velocity}</param>
+          <param name="max_acceleration">${hardware_config.max_acceleration}</param>
+          <param name="max_jerk">${hardware_config.max_jerk}</param>
+          <param name="low_stiffness_mode">${hardware_config.low_stiffness_mode}</param>
+          <param name="low_stiffness_kp">${hardware_config.low_stiffness_kp}</param>
+          <param name="low_stiffness_kd">${hardware_config.low_stiffness_kd}</param>
+          <param name="low_stiffness_torque_bias">${hardware_config.low_stiffness_torque_bias}</param>
+          <param name="use_pinocchio_gravity">${hardware_config.use_pinocchio_gravity}</param>
+          <param name="gravity_feedforward_ratio">${hardware_config.gravity_feedforward_ratio}</param>
+          <param name="use_pinocchio_inverse_dynamics">${hardware_config.use_pinocchio_inverse_dynamics}</param>
+          <param name="urdf_path">${description_package_share}/${hardware_config.urdf_path}</param>
+          <param name="limit_margin">${hardware_config.limit_margin}</param>
+          <param name="limit_stop_margin">${hardware_config.limit_stop_margin}</param>
+          <param name="limit_decel_factor">${hardware_config.limit_decel_factor}</param>
+          <param name="fallback_control_period">${hardware_config.fallback_control_period}</param>
         </xacro:unless>
       </hardware>
@@ -40,6 +51,6 @@
         <param name="position_offset">0.0</param>
         <param name="direction">-1.0</param>
-        <param name="low_stiffness_kp">${low_stiffness_kp_j1}</param>
-        <param name="low_stiffness_kd">${low_stiffness_kd_j1}</param>
+        <param name="low_stiffness_kp">${hardware_config.low_stiffness_kp_j1}</param>
+        <param name="low_stiffness_kd">${hardware_config.low_stiffness_kd_j1}</param>
         <command_interface name="position">
           <!--
@@ -59,5 +70,4 @@
         </command_interface>
         <state_interface name="position"/>
-        <state_interface name="velocity"/>
         <state_interface name="effort"/>
       </joint>
@@ -67,6 +77,6 @@
         <param name="position_offset">0.0</param>
         <param name="direction">1.0</param>
-        <param name="low_stiffness_kp">${low_stiffness_kp_j2}</param>
-        <param name="low_stiffness_kd">${low_stiffness_kd_j2}</param>
+        <param name="low_stiffness_kp">${hardware_config.low_stiffness_kp_j2}</param>
+        <param name="low_stiffness_kd">${hardware_config.low_stiffness_kd_j2}</param>
         <command_interface name="position">
           <!--
@@ -86,5 +96,4 @@
         </command_interface>
         <state_interface name="position"/>
-        <state_interface name="velocity"/>
         <state_interface name="effort"/>
       </joint>
@@ -94,6 +103,6 @@
         <param name="position_offset">0.0</param>
         <param name="direction">-1.0</param>
-        <param name="low_stiffness_kp">${low_stiffness_kp_j3}</param>
-        <param name="low_stiffness_kd">${low_stiffness_kd_j3}</param>
+        <param name="low_stiffness_kp">${hardware_config.low_stiffness_kp_j3}</param>
+        <param name="low_stiffness_kd">${hardware_config.low_stiffness_kd_j3}</param>
         <command_interface name="position">
           <!--
@@ -113,5 +122,4 @@
         </command_interface>
         <state_interface name="position"/>
-        <state_interface name="velocity"/>
         <state_interface name="effort"/>
       </joint>
@@ -121,6 +129,6 @@
         <param name="position_offset">0.0</param>
         <param name="direction">-1.0</param>
-        <param name="low_stiffness_kp">${low_stiffness_kp_j4}</param>
-        <param name="low_stiffness_kd">${low_stiffness_kd_j4}</param>
+        <param name="low_stiffness_kp">${hardware_config.low_stiffness_kp_j4}</param>
+        <param name="low_stiffness_kd">${hardware_config.low_stiffness_kd_j4}</param>
         <command_interface name="position">
           <!--
@@ -140,5 +148,4 @@
         </command_interface>
         <state_interface name="position"/>
-        <state_interface name="velocity"/>
         <state_interface name="effort"/>
       </joint>

Commit message: camera tf (untested)

File: rc_moveit/rc_arm_description/urdf/rc_arm_2/rc_arm_2.urdf.xacro (robot description, xacro)
@@ -211,5 +211,5 @@
   <joint name="camera_d435_link_to_optical_frame" type="fixed">
     <!-- Placeholder optical frame; verify against the RealSense driver TF before using camera data. -->
-    <origin xyz="-0.01 0 0" rpy="0 0 -1.5707963267948966"/>
+    <origin xyz="-0.01 0 0" rpy="0 0 0"/>
     <parent link="camera_d435_link"/>
     <child link="camera_d435_optical_frame"/>

Commit message: camera tf2 untested

File: rc_moveit/rc_arm_description/urdf/rc_arm_2/rc_arm_2.urdf.xacro (robot description, xacro)
@@ -211,5 +211,5 @@
   <joint name="camera_d435_link_to_optical_frame" type="fixed">
     <!-- Placeholder optical frame; verify against the RealSense driver TF before using camera data. -->
-    <origin xyz="-0.01 0 0" rpy="0 0 0"/>
+    <origin xyz="-0.01 0 0" rpy="0 0 1.5707963267948966"/>
     <parent link="camera_d435_link"/>
     <child link="camera_d435_optical_frame"/>

Commit message: j4 angle auto-adjust

File: rc_moveit/rc_arm_description/urdf/rc_arm_2/rc_arm_2.urdf.xacro (robot description, xacro)
@@ -211,5 +211,5 @@
   <joint name="camera_d435_link_to_optical_frame" type="fixed">
     <!-- Placeholder optical frame; verify against the RealSense driver TF before using camera data. -->
-    <origin xyz="-0.01 0 0" rpy="0 0 1.5707963267948966"/>
+    <origin xyz="-0.01 0 0" rpy="0 0 0"/>
     <parent link="camera_d435_link"/>
     <child link="camera_d435_optical_frame"/>

Commit message: simple

File: rc_moveit/rc_arm_description/urdf/rc_arm_2/rc_arm_2.urdf.xacro (robot description, xacro)
@@ -13,4 +13,11 @@
     <color rgba="0.64706 0.61961 0.58824 1.0"/>
   </material>
+  <!-- Simplified cue-stick geometry for faster loading and lighter self-collision. -->
+  <xacro:property name="base_size" value="0.10 0.10 0.05"/>
+  <xacro:property name="l1_size" value="0.025 0.025 0.07"/>
+  <xacro:property name="l2_size" value="0.025 0.025 0.18"/>
+  <xacro:property name="l3_size" value="0.18 0.025 0.025"/>
+  <xacro:property name="l4_size" value="0.04 0.02 0.02"/>
+  <xacro:property name="camera_visual_size" value="0.06 0.02 0.02"/>
   <link name="world"/>
   <joint name="world_to_base_link" type="fixed">
@@ -34,12 +41,12 @@
       <origin xyz="0 0 0" rpy="0 0 0"/>
       <geometry>
-        <mesh filename="package://rc_arm_description/meshes/rc_arm_2/base_link.STL"/>
+        <box size="${base_size}"/>
       </geometry>
       <material name="light_gray"/>
     </visual>
     <collision>
-      <origin xyz="0 0 0" rpy="0 0 0"/>
-      <geometry>
-        <mesh filename="package://rc_arm_description/meshes/rc_arm_2/base_link.STL"/>
+      <origin xyz="0 0 -0.01" rpy="0 0 0"/>
+      <geometry>
+        <box size="${base_size}"/>
       </geometry>
     </collision>
@@ -58,14 +65,14 @@
     </inertial>
     <visual>
-      <origin xyz="0 0 0" rpy="0 0 0"/>
-      <geometry>
-        <mesh filename="package://rc_arm_description/meshes/rc_arm_2/l1.STL"/>
+      <origin xyz="0 0 -0.035" rpy="0 0 0"/>
+      <geometry>
+        <box size="${l1_size}"/>
       </geometry>
       <material name="dark_gray"/>
     </visual>
     <collision>
-      <origin xyz="0 0 0" rpy="0 0 0"/>
-      <geometry>
-        <mesh filename="package://rc_arm_description/meshes/rc_arm_2/l1.STL"/>
+      <origin xyz="0 0 -0.035" rpy="0 0 0"/>
+      <geometry>
+        <box size="${l1_size}"/>
       </geometry>
     </collision>
@@ -91,14 +98,14 @@
     </inertial>
     <visual>
-      <origin xyz="0 0 0" rpy="0 0 0"/>
-      <geometry>
-        <mesh filename="package://rc_arm_description/meshes/rc_arm_2/l2.STL"/>
+      <origin xyz="0 0 0.15" rpy="0 0 0"/>
+      <geometry>
+        <box size="${l2_size}"/>
       </geometry>
       <material name="dark_gray"/>
     </visual>
     <collision>
-      <origin xyz="0 0 0" rpy="0 0 0"/>
-      <geometry>
-        <mesh filename="package://rc_arm_description/meshes/rc_arm_2/l2.STL"/>
+      <origin xyz="0 0 0.15" rpy="0 0 0"/>
+      <geometry>
+        <box size="${l2_size}"/>
       </geometry>
     </collision>
@@ -124,14 +131,14 @@
     </inertial>
     <visual>
-      <origin xyz="0 0 0" rpy="0 0 0"/>
-      <geometry>
-        <mesh filename="package://rc_arm_description/meshes/rc_arm_2/l3.STL"/>
+      <origin xyz="0.13 0 0" rpy="0 0 0"/>
+      <geometry>
+        <box size="${l3_size}"/>
       </geometry>
       <material name="light_gray"/>
     </visual>
     <collision>
-      <origin xyz="0 0 0" rpy="0 0 0"/>
-      <geometry>
-        <mesh filename="package://rc_arm_description/meshes/rc_arm_2/l3.STL"/>
+      <origin xyz="0.13 0 0" rpy="0 0 0"/>
+      <geometry>
+        <box size="${l3_size}"/>
       </geometry>
     </collision>
@@ -157,14 +164,14 @@
     </inertial>
     <visual>
-      <origin xyz="0 0 0" rpy="0 0 0"/>
-      <geometry>
-        <mesh filename="package://rc_arm_description/meshes/rc_arm_2/l4.STL"/>
+      <origin xyz="0.02 0 0" rpy="0 0 0"/>
+      <geometry>
+        <box size="${l4_size}"/>
       </geometry>
       <material name="light_gray"/>
     </visual>
     <collision>
-      <origin xyz="0 0 0" rpy="0 0 0"/>
-      <geometry>
-        <mesh filename="package://rc_arm_description/meshes/rc_arm_2/l4.STL"/>
+      <origin xyz="0.02 0 0" rpy="0 0 0"/>
+      <geometry>
+        <box size="${l4_size}"/>
       </geometry>
     </collision>
@@ -198,5 +205,5 @@
       <origin xyz="0 0 0" rpy="0 0 0"/>
       <geometry>
-        <mesh filename="package://rc_arm_description/meshes/rc_arm_2/d435.STL"/>
+        <box size="${camera_visual_size}"/>
       </geometry>
       <material name="d435_gray"/>
